File: sch/extram.kicad_sch (KiCad schematic)
At the start: 8 parts

Commit message: More routing, USB iface
Parts:
- added U11: 74AC14, Package_SO:TSSOP-14_4.4x5mm_P0.65mm, symbol 74xx:74HC14
- ERAM0: value (none) -> IS62WV10248; footprint (none) -> Package_SO:TSOP-II-44_10.16x18.41mm_P0.8mm
Connections:
- net +5V: now also U11.14 (VCC)
- net GND: now also U11.7 (GND)
- net ~{ERAM_CS0}: now also U11.1
- net ~{ERAM_CS1}: now also U11.9
- net ~{ERAM_CS2}: now also U11.3
- net ~{ERAM_CS3}: now also U11.5
- net at ERAM3.40 (CS2): now also U11.6
- net at ERAM0.40 (CS2): now also U11.2
- net at ERAM2.40 (CS2): now also U11.4
- net at ERAM1.40 (CS2): now also U11.8
- net BUS_W~{R} renamed ~{BUS_READ}
- net WRITE renamed ~{BUS_WRITE}
Other:
- note added: "0x01000000 - 0x08FFFFFF"
- moved on the sheet: C12, C13, C14, C2, ERAM0, ERAM1, ERAM2, ERAM3
