File: sch/memory.kicad_sch (KiCad schematic)
At the start: 9 parts, among them U8 74AHC00

Commit message: Serial interface
Parts:
- removed AD_DEC1: 74HCT154, Package_SO:SO-24_5.3x15mm_P1.27mm, symbol 74xx:74LS154
- removed C18: 100nF, Capacitor_SMD:C_1206_3216Metric_Pad1.33x1.80mm_HandSolder, symbol Device:C_Small
- removed C22: 10nF, Capacitor_SMD:C_0603_1608Metric, symbol Device:C_Small
- removed U8: 74AHC00, Package_SO:TSSOP-14_4.4x5mm_P0.65mm, symbol 74xx:74HC00
- C15, C16: footprint Capacitor_SMD:C_1206_3216Metric_Pad1.33x1.80mm_HandSolder -> (none)
- R2: footprint Resistor_SMD:R_1206_3216Metric_Pad1.30x1.75mm_HandSolder -> (none)
- RAM1: renamed from SRAM1; footprint Package_DIP:DIP-28_W15.24mm -> Package_DIP:DIP-28_W15.24mm_LongPads
- ROM1: footprint Package_DIP:DIP-28_W15.24mm_LongPads -> Package_DIP:DIP-28_W15.24mm_Socket_LongPads
Connections:
- no-connect marks 1 -> 0
Other:
- removed sheet ERAM
- note removed: "Address Decoder"
- note removed: "Currently nothing is connected here so data in this range will be written onto thin air"
- note removed: "ERAM: 0x100000 - 0x8FFFFF"
- note removed: "IO: 0x010000 - 0x0FFFFF"
- note removed: "PAGE 0: ROM and Stack RAM ~{ } RAM: 0x0000 - 0x7FFF ROM: 0x8000 - 0xFFFF"
- note removed: "PRP: 0xB00000 - 0xFFFFFF"
- note removed: "VID: 0x900000 - 0xAFFFFF"
- note removed: "ZERO: 0x000000 - 0x0FFFFF"
- company: (none) -> zrthxn
- title: (none) -> 8puter
- moved on the sheet: C15, C16, R2, RAM1, ROM1

Commit message: Serial, debug and prph headers
Parts:
- C15, C16: footprint (none) -> Capacitor_SMD:C_0805_2012Metric
- R2: footprint (none) -> Resistor_SMD:R_0805_2012Metric
Changed lines of the file:
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@@
       (effects (font (size 1.27 1.27)) (justify left))
     )
-    (property "Footprint" "" (id 2) (at 154.178 140.335 90)
+    (property "Footprint" "Resistor_SMD:R_0805_2012Metric" (id 2) (at 154.178 140.335 90)
       (effects (font (size 1.27 1.27)) hide)
     )
@@
     (property "Reference" "C15" (id 0) (at 111.125 93.345 90))
     (property "Value" "100nF" (id 1) (at 104.775 93.345 90))
-    (property "Footprint" "" (id 2) (at 108.585 95.885 0)
+    (property "Footprint" "Capacitor_SMD:C_0805_2012Metric" (id 2) (at 108.585 95.885 0)
       (effects (font (size 1.27 1.27)) hide)
     )
@@
     (property "Reference" "C16" (id 0) (at 111.125 31.115 90))
     (property "Value" "100nF" (id 1) (at 104.775 31.115 90))
-    (property "Footprint" "" (id 2) (at 108.585 33.655 0)
+    (property "Footprint" "Capacitor_SMD:C_0805_2012Metric" (id 2) (at 108.585 33.655 0)
       (effects (font (size 1.27 1.27)) hide)
     )
