File: sch/memory.kicad_sch (KiCad schematic)
At the start: 6 parts

Commit message: small updates
Parts:
- ROM_WRITE1: value (none) -> Conn_01x03; footprint (none) -> Connector_PinHeader_2.54mm:PinHeader_1x03_P2.54mm_Vertical
Changed lines of the file:
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@@
     (effects (font (size 1.8 1.8)) (justify left bottom))
   )
+  (text "System Memory" (at 31.75 26.035 0)
+    (effects (font (size 2 2) (thickness 0.254) bold) (justify left bottom))
+  )
   (text "Tying A14 to ~{OE} and \nchip's A14 to GND makes the RAM\neffectively 16K bytes size, \nwith upper half in use."
-    (at 121.92 99.695 0)
+    (at 123.825 99.695 0)
     (effects (font (size 1.27 1.27)) (justify left bottom))
   )
@@
     (effects (font (size 1.27 1.27)) (justify left bottom))
   )
-  (text "System Memory" (at 31.75 25.4 0)
-    (effects (font (size 2 2) (thickness 0.4) bold) (justify left bottom))
-  )
   (label "D2" (at 66.04 117.475 180)
     (effects (font (size 1.27 1.27)) (justify right bottom))
@@
       (effects (font (size 1.27 1.27)) (justify left))
     )
-    (property "Value" "" (id 1) (at 136.525 154.3049 0)
-      (effects (font (size 1.27 1.27)) (justify left))
-    )
-    (property "Footprint" "" (id 2) (at 133.985 153.035 0)
-      (effects (font (size 1.27 1.27)) hide)
-    )
+    (property "Value" "Conn_01x03" (id 1) (at 136.525 154.3049 0)
+      (effects (font (size 1.27 1.27)) (justify left))
+    )
+    (property "Footprint" "Connector_PinHeader_2.54mm:PinHeader_1x03_P2.54mm_Vertical" (id 2) (at 133.985 153.035 0)
+      (effects (font (size 1.27 1.27)) hide)
+    )
