File: sch/serial.kicad_sch (KiCad schematic)
At the start: 4 parts

Commit message: Serial, debug and prph headers
Parts:
- removed SERIAL1: (no value), symbol Connector_Generic:Conn_2Rows-11Pins
- added C13: 30pF, Capacitor_SMD:C_0805_2012Metric, symbol Device:C_Small
- added R4: 1M, Resistor_THT:R_Axial_DIN0204_L3.6mm_D1.6mm_P7.62mm_Horizontal, symbol Device:R
- added SERIAL1: Conn_02x05_Odd_Even, Connector_PinHeader_2.54mm:PinHeader_2x05_P2.54mm_Vertical, symbol Connector_Generic:Conn_02x05_Odd_Even
- added Y1: 1.8432MHz, Crystal:Crystal_HC49-4H_Vertical, symbol Device:Crystal
- C10, C12: value (none) -> 100nF; footprint (none) -> Capacitor_SMD:C_0805_2012Metric
- SERC1: value (none) -> W65C51NxQ; footprint (none) -> Package_QFP:LQFP-32_7x7mm_P0.8mm
Connections:
- net +5V: now also SERIAL1.2 (Pin_2)
- net GND: now also C13.2, SERIAL1.10 (Pin_10)
- net at SERC1.1 (RxC): now also SERIAL1.8 (Pin_8)
- net at SERC1.14 (~{DCD}): now also SERIAL1.9 (Pin_9)
- net at SERC1.15 (~{DSR}): now also SERIAL1.7 (Pin_7)
- net at SERC1.2 (XTAL1): now also R4.1, Y1.2
- net at SERC1.3 (XTAL2): now also C13.1, R4.2, Y1.1
- net at SERC1.4 (~{RTS}): now also SERIAL1.1 (Pin_1)
- net at SERC1.5 (~{CTS}): now also SERIAL1.3 (Pin_3)
- net at SERC1.6 (TxD): now also SERIAL1.6 (Pin_6)
- net at SERC1.7 (~{DTR}): now also SERIAL1.5 (Pin_5)
- net at SERC1.9 (RxD): now also SERIAL1.4 (Pin_4)
Other:
- moved on the sheet: C10, C12, SERC1
