File: sch/power.kicad_sch (KiCad schematic)
At the start: 6 parts, among them SW1 RESET_SW, U6 MAX811MEUS-T

Commit message: Pivot to 6502
Parts:
- added C19, C20: 100nF, Capacitor_THT:CP_Radial_D5.0mm_P2.00mm, symbol Device:C_Polarized_Small
- added C5, C6: 10uF, Capacitor_THT:CP_Radial_D5.0mm_P2.00mm, symbol Device:C_Polarized_Small
- added C7, C8: 1uF, Capacitor_THT:CP_Radial_D5.0mm_P2.00mm, symbol Device:C_Polarized_Small
- added FB1, FB2: FerriteBead_Small, symbol Device:FerriteBead_Small
- added PWREG1: LT1962-3.3, Package_SO:MSOP-8_3x3mm_P0.65mm, symbol Regulator_Linear:LT1962-3.3
- C1: value 1uF -> 10uF
Connections:
- net 3.3V: now also FB1.1
- net 5V: now also FB2.1; no longer C17.1, PWREG2.1 (OUT)
- net GND: now also C19.2, C20.2, C5.2, C6.2, C7.2, C8.2
- net PWR: now also C5.1, PWREG1.8 (IN)
- new net: C19.1, C6.1, C7.1, FB1.2, PWREG1.1 (OUT)
- new net: C17.1, C20.1, C8.1, FB2.2, PWREG2.1 (OUT)
- no-connect marks 2 -> 3
Other:
- moved on the sheet: C11, C17, SW1, U6

Commit message: Serial interface
Parts:
- removed FB1: FerriteBead_Small, symbol Device:FerriteBead_Small
- C11: footprint Capacitor_SMD:C_1206_3216Metric_Pad1.33x1.80mm_HandSolder -> (none)
- C17, C19, C20, C6, C7, C8: footprint Capacitor_THT:CP_Radial_D5.0mm_P2.00mm -> (none)
- RESET_SW1: renamed from SW1; value RESET_SW -> (none)
Connections:
- net 3.3V: now also C19.1, C6.1, C7.1, PWREG1.1 (OUT)
- net 5V: now also C5.1, PWREG1.8 (IN)
- net GND: now also PWREG1.4 (GND)
- net PWR: no longer C5.1, PWREG1.8 (IN)
- net RST renamed ~{RST}
Other:
- company: (none) -> zrthxn
- title: (none) -> 8puter
- moved on the sheet: C1, C11, C17, C19, C20, C5, C6, C7, C8, FB2, PWREG1, PWREG2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

Commit message: Serial, debug and prph headers
Parts:
- removed C5: 10uF, Capacitor_THT:CP_Radial_D5.0mm_P2.00mm, symbol Device:C_Polarized_Small
- removed FB2: FerriteBead_Small, symbol Device:FerriteBead_Small
- C11, C17, C19, C20, C6, C7, C8: footprint (none) -> Capacitor_SMD:C_0805_2012Metric
- RESET_SW1: value (none) -> PUSHBTN
Connections:
- net 5V: now also C17.1, C20.1, C8.1, PWREG2.1 (OUT)
- no-connect marks 3 -> 2
Changed lines of the file:
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@@
   (junction (at 152.4 102.235) (diameter 0) (color 0 0 0 0)
-  )
-  (junction (at 114.3 102.235) (diameter 0) (color 0 0 0 0)
   )
   (junction (at 152.4 71.12) (diameter 0) (color 0 0 0 0)
@@
   (no_connect (at 124.46 78.74))
   (no_connect (at 144.78 78.74))
-  (no_connect (at 188.595 33.02))
   (wire (pts (xy 162.56 102.235) (xy 152.4 102.235))
     (stroke (width 0) (type default) (color 0 0 0 0))
   )
-  (wire (pts (xy 194.945 71.12) (xy 187.325 71.12))
-    (stroke (width 0) (type default) (color 0 0 0 0))
-  )
   (wire (pts (xy 172.085 71.12) (xy 162.56 71.12))
     (stroke (width 0) (type default) (color 0 0 0 0))
@@
     (stroke (width 0) (type default) (color 0 0 0 0))
   )
-  (wire (pts (xy 114.3 102.235) (xy 124.46 102.235))
-    (stroke (width 0) (type default) (color 0 0 0 0))
-  )
   (wire (pts (xy 162.56 71.12) (xy 152.4 71.12))
     (stroke (width 0) (type default) (color 0 0 0 0))
@@
     (stroke (width 0) (type default) (color 0 0 0 0))
   )
-  (wire (pts (xy 107.315 102.235) (xy 114.3 102.235))
+  (wire (pts (xy 107.315 102.235) (xy 124.46 102.235))
     (stroke (width 0) (type default) (color 0 0 0 0))
   )
@@
     (stroke (width 0) (type default) (color 0 0 0 0))
   )
-  (wire (pts (xy 188.595 33.02) (xy 194.945 33.02))
-    (stroke (width 0) (type default) (color 0 0 0 0))
-  )
   (wire (pts (xy 100.965 136.525) (xy 100.965 144.145))
     (stroke (width 0) (type default) (color 0 0 0 0))
@@
     (stroke (width 0) (type default) (color 0 0 0 0))
   )
-  (wire (pts (xy 172.085 102.235) (xy 194.945 102.235))
+  (wire (pts (xy 172.085 102.235) (xy 184.15 102.235))
     (stroke (width 0) (type default) (color 0 0 0 0))
   )
@@
     (stroke (width 0) (type default) (color 0 0 0 0))
   )
-  (wire (pts (xy 114.3 102.235) (xy 114.3 104.775))
-    (stroke (width 0) (type default) (color 0 0 0 0))
-  )
   (wire (pts (xy 172.085 102.235) (xy 162.56 102.235))
     (stroke (width 0) (type default) (color 0 0 0 0))
@@
     (stroke (width 0) (type default) (color 0 0 0 0))
   )
-  (wire (pts (xy 182.245 71.12) (xy 172.085 71.12))
+  (wire (pts (xy 172.085 71.12) (xy 184.15 71.12))
     (stroke (width 0) (type default) (color 0 0 0 0))
   )
@@
     (effects (font (size 1.27 1.27)) (justify left))
   )
-  (hierarchical_label "12V" (shape output) (at 194.945 33.02 0)
-    (effects (font (size 1.27 1.27)) (justify left))
-  )
-  (hierarchical_label "5V" (shape output) (at 194.945 71.12 0)
+  (hierarchical_label "5V" (shape output) (at 184.15 71.12 0)
     (effects (font (size 1.27 1.27)) (justify left))
   )
@@
     (effects (font (size 1.27 1.27)) (justify right))
   )
-  (hierarchical_label "3.3V" (shape output) (at 194.945 102.235 0)
+  (hierarchical_label "3.3V" (shape output) (at 184.15 102.235 0)
     (effects (font (size 1.27 1.27)) (justify left))
   )
@@
     (pin "8")
   )
-  (symbol (lib_id "Device:FerriteBead_Small") (at 184.785 71.12 270) (unit 1)
-    (in_bom yes) (on_board yes) (fields_autoplaced)
-    (property "Reference" "FB2" (id 0) (at 184.8231 64.77 90))
-    (property "Value" "FerriteBead_Small" (id 1) (at 184.8231 67.31 90))
-    (property "Footprint" "" (id 2) (at 184.785 69.342 90)
-      (effects (font (size 1.27 1.27)) hide)
-    )
-    (property "Datasheet" "~" (id 3) (at 184.785 71.12 0)
-      (effects (font (size 1.27 1.27)) hide)
-    )
-    (pin "1")
-    (pin "2")
-  )
   (symbol (lib_id "Device:C_Polarized_Small") (at 172.085 107.315 0) (mirror y) (unit 1)
     (in_bom yes) (on_board yes)
@@
       (effects (font (size 1.27 1.27)) (justify right))
     )
-    (property "Footprint" "" (id 2) (at 172.085 107.315 0)
+    (property "Footprint" "Capacitor_SMD:C_0805_2012Metric" (id 2) (at 172.085 107.315 0)
       (effects (font (size 1.27 1.27)) hide)
     )
@@
       (effects (font (size 1.27 1.27)) (justify right))
     )
-    (property "Footprint" "" (id 2) (at 152.4 107.315 0)
+    (property "Footprint" "Capacitor_SMD:C_0805_2012Metric" (id 2) (at 152.4 107.315 0)
       (effects (font (size 1.27 1.27)) hide)
     )
@@
       (effects (font (size 1.27 1.27)) (justify left))
     )
-    (property "Footprint" "" (id 2) (at 117.1702 144.145 0)
+    (property "Footprint" "Capacitor_SMD:C_0805_2012Metric" (id 2) (at 117.1702 144.145 0)
       (effects (font (size 1.27 1.27)) hide)
     )
@@
       (effects (font (size 1.27 1.27)) (justify right))
     )
-    (property "Footprint" "" (id 2) (at 162.56 107.315 0)
+    (property "Footprint" "Capacitor_SMD:C_0805_2012Metric" (id 2) (at 162.56 107.315 0)
       (effects (font (size 1.27 1.27)) hide)
     )
@@
       (effects (font (size 1.27 1.27)) (justify right))
     )
-    (property "Footprint" "" (id 2) (at 172.085 76.2 0)
+    (property "Footprint" "Capacitor_SMD:C_0805_2012Metric" (id 2) (at 172.085 76.2 0)
       (effects (font (size 1.27 1.27)) hide)
     )
@@
     (pin "1")
   )
-  (symbol (lib_id "Device:C_Polarized_Small") (at 114.3 107.315 0) (unit 1)
-    (in_bom yes) (on_board yes)
-    (property "Reference" "C5" (id 0) (at 109.22 106.045 0)
-      (effects (font (size 1.27 1.27)) (justify left))
-    )
-    (property "Value" "10uF" (id 1) (at 111.76 108.585 0)
-      (effects (font (size 1.27 1.27)) (justify right))
-    )
-    (property "Footprint" "Capacitor_THT:CP_Radial_D5.0mm_P2.00mm" (id 2) (at 114.3 107.315 0)
-      (effects (font (size 1.27 1.27)) hide)
-    )
-    (property "Datasheet" "~" (id 3) (at 114.3 107.315 0)
-      (effects (font (size 1.27 1.27)) hide)
-    )
-    (pin "1")
-    (pin "2")
-  )
   (symbol (lib_id "power:GND") (at 134.62 114.935 0) (unit 1)
     (in_bom yes) (on_board yes) (fields_autoplaced)
@@
       (effects (font (size 1.27 1.27)) hide)
     )
-    (property "Value" "" (id 1) (at 134.62 119.38 0))
+    (property "Value" "GND" (id 1) (at 134.62 119.38 0))
     (property "Footprint" "" (id 2) (at 134.62 114.935 0)
       (effects (font (size 1.27 1.27)) hide)
@@
       (effects (font (size 1.27 1.27)) (justify right))
     )
-    (property "Footprint" "" (id 2) (at 162.56 76.2 0)
+    (property "Footprint" "Capacitor_SMD:C_0805_2012Metric" (id 2) (at 162.56 76.2 0)
       (effects (font (size 1.27 1.27)) hide)
     )
@@
     (in_bom yes) (on_board yes)
     (property "Reference" "RESET_SW1" (id 0) (at 107.315 139.065 0))
-    (property "Value" "" (id 1) (at 107.315 141.605 0))
+    (property "Value" "PUSHBTN" (id 1) (at 107.315 141.605 0))
     (property "Footprint" "Button_Switch_THT:SW_PUSH_6mm_H13mm" (id 2) (at 107.315 131.445 0)
       (effects (font (size 1.27 1.27)) hide)
@@
       (effects (font (size 1.27 1.27)) (justify right))
     )
-    (property "Footprint" "" (id 2) (at 152.4 76.2 0)
+    (property "Footprint" "Capacitor_SMD:C_0805_2012Metric" (id 2) (at 152.4 76.2 0)
       (effects (font (size 1.27 1.27)) hide)
     )
@@
     (pin "2")
   )
-  (symbol (lib_id "power:GND") (at 114.3 109.855 0) (unit 1)
-    (in_bom yes) (on_board yes) (fields_autoplaced)
-    (property "Reference" "#PWR0140" (id 0) (at 114.3 116.205 0)
-      (effects (font (size 1.27 1.27)) hide)
-    )
-    (property "Value" "GND" (id 1) (at 114.3 114.935 0))
-    (property "Footprint" "" (id 2) (at 114.3 109.855 0)
-      (effects (font (size 1.27 1.27)) hide)
-    )
-    (property "Datasheet" "" (id 3) (at 114.3 109.855 0)
-      (effects (font (size 1.27 1.27)) hide)
-    )
-    (pin "1")
-  )
   (sheet_instances

Commit message: First completed routing
Parts:
- removed C19, C20: 100nF, Capacitor_SMD:C_0805_2012Metric, symbol Device:C_Polarized_Small
- removed PWREG1: LT1962-3.3, Package_SO:MSOP-8_3x3mm_P0.65mm, symbol Regulator_Linear:LT1962-3.3
- removed PWREG2: LT1962-5, Package_SO:MSOP-8_3x3mm_P0.65mm, symbol Regulator_Linear:LT1962-5
- added C14, C5: (no value), symbol Device:C_Small
- added C19, C20: (no value), Capacitor_SMD:C_0805_2012Metric, symbol Device:C_Small
- added D1: (no value), symbol Device:LED
- added R29: (no value), symbol Device:R
- added REG1, REG2, REG3: (no value), symbol Regulator_Linear:NCP1117-5.0_SOT223
- C1: value 10uF -> (none); footprint Capacitor_THT:CP_Radial_D5.0mm_P2.00mm -> (none); symbol Device:C_Polarized_Small -> Device:C_Small
- C11: symbol Device:C -> Device:C_Small
- C17, C6: value 10uF -> (none); symbol Device:C_Polarized_Small -> Device:C_Small
- C7, C8: value 1uF -> (none); symbol Device:C_Polarized_Small -> Device:C_Small
Connections:
- net 3.3V: now also REG2.2 (VO)
- net 5V: now also C14.1, C5.1, REG1.2 (VO), REG2.3 (VI), REG3.3 (VI)
- net GND: now also C14.2, C19.2, C20.2, C5.2, R29.2, REG1.1 (GND), REG2.1 (GND), REG3.1 (GND)
- net PWR: now also D1.2 (A), REG1.3 (VI)
- new net: D1.1 (K), R29.1
- new net 3V: C19.1, C20.1, REG3.2 (VO)
- no-connect marks 2 -> 0
Other:
- note added: "FPGA supply"
- note added: "Main board supply"
- note added: "RESET BUTTON"
- note added: "STM32 supply"
- moved on the sheet: C11, RESET_SW1, U6
