File: sch/video.kicad_sch (KiCad schematic)
At the start: 4 parts

Commit message: serial rollback
Connections:
- net +3V0: no longer C23.1, VIDEO1.1 (VBAT), VIDEO1.24 (VDD), VIDEO1.36 (VDD), VIDEO1.48 (VDD), VIDEO1.9 (VDDA)
- net A11: now reaches VIDEO1.46 (PB9)
- new net +3V3: C23.1, VIDEO1.1 (VBAT), VIDEO1.24 (VDD), VIDEO1.36 (VDD), VIDEO1.48 (VDD), VIDEO1.9 (VDDA)
Other:
- note added: "0x4800 - 0x480F"
Changed lines of the file:
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@@
     (company "zrthxn")
   )
+  (junction (at 139.7 140.335) (diameter 0) (color 0 0 0 0)
+  )
+  (junction (at 85.09 107.315) (diameter 0) (color 0 0 0 0)
+  )
+  (junction (at 162.56 84.455) (diameter 0) (color 0 0 0 0)
+  )
+  (junction (at 140.97 140.335) (diameter 0) (color 0 0 0 0)
+  )
+  (junction (at 85.09 89.535) (diameter 0) (color 0 0 0 0)
+  )
+  (junction (at 144.78 64.135) (diameter 0) (color 0 0 0 0)
+  )
+  (junction (at 104.775 109.855) (diameter 0) (color 0 0 0 0)
+  )
+  (junction (at 85.09 94.615) (diameter 0) (color 0 0 0 0)
+  )
+  (junction (at 142.24 140.335) (diameter 0) (color 0 0 0 0)
+  )
+  (junction (at 142.24 64.135) (diameter 0) (color 0 0 0 0)
+  )
+  (junction (at 139.7 64.135) (diameter 0) (color 0 0 0 0)
+  )
   (junction (at 142.24 59.055) (diameter 0) (color 0 0 0 0)
-  )
-  (junction (at 139.7 140.335) (diameter 0) (color 0 0 0 0)
-  )
-  (junction (at 85.09 107.315) (diameter 0) (color 0 0 0 0)
-  )
-  (junction (at 162.56 84.455) (diameter 0) (color 0 0 0 0)
-  )
-  (junction (at 140.97 140.335) (diameter 0) (color 0 0 0 0)
-  )
-  (junction (at 85.09 89.535) (diameter 0) (color 0 0 0 0)
-  )
-  (junction (at 144.78 64.135) (diameter 0) (color 0 0 0 0)
-  )
-  (junction (at 104.775 109.855) (diameter 0) (color 0 0 0 0)
-  )
-  (junction (at 85.09 94.615) (diameter 0) (color 0 0 0 0)
-  )
-  (junction (at 142.24 140.335) (diameter 0) (color 0 0 0 0)
-  )
-  (junction (at 142.24 64.135) (diameter 0) (color 0 0 0 0)
-  )
-  (junction (at 139.7 64.135) (diameter 0) (color 0 0 0 0)
   )
   (junction (at 85.09 84.455) (diameter 0) (color 0 0 0 0)
@@
     (stroke (width 0) (type default) (color 0 0 0 0))
   )
+  (bus_entry (at 116.205 117.475) (size 2.54 2.54)
+    (stroke (width 0) (type default) (color 0 0 0 0))
+  )
   (bus_entry (at 119.38 97.155) (size 2.54 2.54)
     (stroke (width 0) (type default) (color 0 0 0 0))
@@
     (stroke (width 0) (type default) (color 0 0 0 0))
   )
+  (bus (pts (xy 115.57 117.475) (xy 116.205 117.475))
+    (stroke (width 0) (type default) (color 0 0 0 0))
+  )
+  (wire (pts (xy 118.745 120.015) (xy 124.46 120.015))
+    (stroke (width 0) (type default) (color 0 0 0 0))
+  )
   (wire (pts (xy 160.02 104.775) (xy 157.48 104.775))
     (stroke (width 0) (type default) (color 0 0 0 0))
   )
+  (text "0x4800 - 0x480F" (at 31.75 28.575 0)
+    (effects (font (size 1.27 1.27)) (justify left bottom))
+  )
   (text "Video will be generated using a \nmicrocontroller which is fast enough to \ngenerate the VGA timing signals.\n\nCPU will send a single byte to the MCU which can\nbe be a char code or index of glyph, and the MCU\njust generates the video signal.\n\nThis setup is limited in generating graphics but\nit avoids having to keep a large framebuffer."
-    (at 31.75 52.705 0)
+    (at 31.75 60.325 0)
     (effects (font (size 1.27 1.27)) (justify left bottom))
   )
@@
     (effects (font (size 1.27 1.27)) (justify left bottom))
   )
+  (label "A11" (at 120.65 120.015 0)
+    (effects (font (size 1.27 1.27)) (justify left bottom))
+  )
   (label "D6" (at 157.48 107.315 0)
     (effects (font (size 1.27 1.27)) (justify left bottom))
@@
   )
   (hierarchical_label "~{VID_CS}" (shape input) (at 124.46 122.555 180)
+    (effects (font (size 1.27 1.27)) (justify right))
+  )
+  (hierarchical_label "A[0..15]" (shape input) (at 115.57 117.475 180)
     (effects (font (size 1.27 1.27)) (justify right))
   )
@@
     (pin "1")
   )
+  (symbol (lib_id "power:+3.3V") (at 142.24 59.055 0) (unit 1)
+    (in_bom yes) (on_board yes) (fields_autoplaced)
+    (property "Reference" "#PWR023" (id 0) (at 142.24 62.865 0)
+      (effects (font (size 1.27 1.27)) hide)
+    )
+    (property "Value" "+3.3V" (id 1) (at 142.24 53.34 0))
+    (property "Footprint" "" (id 2) (at 142.24 59.055 0)
+      (effects (font (size 1.27 1.27)) hide)
+    )
+    (property "Datasheet" "" (id 3) (at 142.24 59.055 0)
+      (effects (font (size 1.27 1.27)) hide)
+    )
+    (pin "1")
+  )
   (symbol (lib_id "power:GND") (at 160.02 66.675 0) (unit 1)
     (in_bom yes) (on_board yes)
@@
       (effects (font (size 1.27 1.27)) hide)
     )
-    (pin "1")
-  )
-  (symbol (lib_id "power:+3V0") (at 142.24 59.055 0) (unit 1)
-    (in_bom yes) (on_board yes)
-    (property "Reference" "#PWR0136" (id 0) (at 142.24 62.865 0)
-      (effects (font (size 1.27 1.27)) hide)
-    )
-    (property "Value" "+3V0" (id 1) (at 143.51 57.15 0)
-      (effects (font (size 1.27 1.27)) (justify left))
-    )
-    (property "Footprint" "" (id 2) (at 142.24 59.055 0)
-      (effects (font (size 1.27 1.27)) hide)
-    )
-    (property "Datasheet" "" (id 3) (at 142.24 59.055 0)
-      (effects (font (size 1.27 1.27)) hide)
-    )
