File: 8puter.kicad_pcb (KiCad board)
At the start: 2 copper layers, 100 x 100 mm, 111 parts, among them J1 PWR-DC, U1 74AC00, U2 74AHC74, U3 74HC126, U6 MAX811TEUS+T, X1 ECS-2200BX-100

Commit message: KiCad v7
Other:
- board text removed: "POWER OFF before changing"

Commit message: Board Revision
Parts:
- moved C2 4.12 mm to (152.0, 88.4), turned to 180 degrees
- moved R24 2.81 mm to (152.0, 121.8)
- moved R19 2.63 mm to (152.0, 109.0)
- moved R22 2.59 mm to (152.0, 116.7)
- moved R13 2.57 mm to (152.0, 93.7)
- moved R20 2.57 mm to (152.0, 111.6)
- moved R23 2.55 mm to (152.0, 119.3)
- moved R21 2.53 mm to (152.0, 114.2)
- moved R14 2.51 mm to (152.0, 96.4)
- moved R17 2.49 mm to (152.0, 104.0)
- moved R15 2.47 mm to (152.0, 98.9)
- moved R18 2.45 mm to (152.0, 106.6)
- moved R16 2.43 mm to (152.0, 101.5)
- moved C4 1.67 mm to (152.0, 91.2), turned to 180 degrees
Routing:
- net +5V: track 165.1 -> 163.3 mm, vias 9 -> 8
- net ADDR11: track 197.6 -> 197.1 mm
- net GND: vias 23 -> 22
